File: esquematico-de-incubadora/esquematico-de-incubadora.kicad_pcb (KiCad board)
At the start: 2 copper layers, 51.9 x 55.8 mm, 26 parts, among them J1 Cable_PAD, J2 LCD, J3 LCD, J4 Cable_PAD, J5 Conn_01x02, J8 Conn_01x02, Q1 IRFZ44N, Q2 IRFZ44N, SW1 SW_Push, U2 PC817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

Commit message: modificacion
Parts:
- moved Q1 2.57 mm to (185.5, 84.6), turned to -90 degrees
- moved Q2 2.51 mm to (185.8, 68.6), turned to -90 degrees
- moved D2 1.08 mm to (178.0, 79.5)
- moved R6 1.06 mm to (176.0, 84.6)
- moved D1 1.06 mm to (177.3, 89.9)
Connections:
- D1 pad 2: +3.3V -> +5V
- D2 pad 2: +3.3V -> +5V
- ESP32_36PINES1 pad 6: unconnected-(ESP32_36PINES1-IO35-Pad6) -> DHT11
- ESP32_36PINES1 pad 7: DHT11 -> cooler
- ESP32_36PINES1 pad 8: unconnected-(ESP32_36PINES1-IO33-Pad8) -> resistencia
- J8 pad 2: +3.3V -> +5V
- Q1 pad 2: GND -> Net-(D2-A)
- Q1 pad 3: Net-(D2-A) -> GND
- Q2 pad 2: GND -> Net-(D3-A)
- Q2 pad 3: Net-(D3-A) -> GND
- U2 pad 4: +3.3V -> +5V
Routing:
- net +5V: track 54.0 -> 107.3 mm
- net +3.3V: track 72.1 -> 30.8 mm
- net cooler: track 3.75 -> 29.1 mm
- net resistencia: track 3.70 -> 20.9 mm
- net Net-(Q1-G): track 4.32 -> 9.63 mm
- net Net-(Q2-G): track 4.27 -> 9.43 mm
- net DHT11: track 17.6 -> 14.9 mm
- net Net-(D2-A): track 23.8 -> 25.5 mm
- net Net-(J4-Pad1): track 6.73 -> 7.52 mm
