File: esquematico-de-incubadora/esquematico-de-incubadora.kicad_sch (KiCad schematic)
At the start: 26 parts, among them J1 Cable_PAD, J2 LCD, J3 LCD, J4 Cable_PAD, J5 Conn_01x02, J8 Conn_01x02, Q1 IRFZ44N, Q2 IRFZ44N, SW1 SW_Push, U2 PC817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

Commit message: modificacion
Connections:
- net +3.3V: no longer D1.2 (A), D2.2 (K), J8.2 (Pin_2), U2.4
- net +5V: now also D1.2 (A), D2.2 (K), J8.2 (Pin_2), U2.4
- net DHT11: now also ESP32_36PINES1.6 (IO35); no longer ESP32_36PINES1.7 (IO32)
- net GND: now also Q1.3 (S), Q2.3 (S); no longer Q1.2 (D), Q2.2 (D)
- net cooler: now also ESP32_36PINES1.7 (IO32); no longer ESP32_36PINES1.13 (IO12)
- net resistencia: now also ESP32_36PINES1.8 (IO33); no longer ESP32_36PINES1.12 (IO14)
- net at D3.1 (A), J5.1 (Pin_1), R3.1: now also Q2.2 (D); no longer Q2.3 (S)
- net at D2.1 (A), J8.1 (Pin_1), R6.1: now also Q1.2 (D); no longer Q1.3 (S)
Other:
- moved on the sheet: Q1, Q2
